File: LandingGearSchematic_3.sch (EAGLE design)
At the start: 76 parts, among them J1 3x2 M, J2 S2B-PH-SM4-TB(LF)(SN), J3 629105136821, SW1 AYZ0202AGRLC, SW2 !RESET, U1 MCP73831, U2 MIC5219, U3 ATMEGA32U4-AUR, X2 16 MHz

Commit message: REV 3
Connections:
- net N$11 renamed NC_D11_R
- net N$12 renamed NC_D6_R
- net N$17 renamed NC_D4_R
- net N$18 renamed NC_D2_R
- net N$21 renamed NC_D0_R
- net N$23 renamed NC_A3_R
- net N$24 renamed NC_A1_R
- net N$25 renamed NC_A4_R
- net N$26 renamed NC_A2_R
- net N$27 renamed NC_A0_R
- net ND_D5 renamed ND_D5_R
- removed net N$2: R9.2
- removed net N$5: R13.2
- removed net N$6: R14.2
- removed net N$8: R15.2
- removed net N$9: R16.2
- new net NC_D12_R: R9.1, SV2.10
- new net NC_D1_R: R16.1, SV2.2
- new net NC_D3_R: R15.1, SV2.4
- new net NC_D7_R: R13.1, SV2.8
- net NC_D1: now also R16.2; no longer R16.1, SV2.2
- net NC_D12: now also R9.2; no longer R9.1, SV2.10
- net NC_D3: now also R15.2; no longer R15.1, SV2.4
- net NC_D5: now also R14.2
- net NC_D7: now also R13.2; no longer R13.1, SV2.8
Changed lines of the file:
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@@
+</segment>
+</net>
+<net name="ND_D5_R" class="0">
+<segment>
+<pinref part="SV2" gate="1" pin="6"/>
+<wire x1="172.72" y1="104.14" x2="162.56" y2="104.14" width="0.1524" layer="91"/>
+<pinref part="R14" gate="G$1" pin="1"/>
+</segment>
+</net>
+<net name="NC_D11" class="0">
+<segment>
+<label x="218.44" y="109.22" size="1.27" layer="95" xref="yes"/>
+<wire x1="205.74" y1="109.22" x2="218.44" y2="109.22" width="0.1524" layer="91"/>
+<pinref part="R18" gate="G$1" pin="1"/>
+</segment>
+</net>
+<net name="N$1" class="0">
+<segment>
+<pinref part="SV2" gate="1" pin="12"/>
+<wire x1="172.72" y1="111.76" x2="162.56" y2="111.76" width="0.1524" layer="91"/>
+<pinref part="R7" gate="G$1" pin="1"/>
+</segment>
+</net>
+<net name="NC_D7" class="0">
+<segment>
+<wire x1="152.4" y1="106.68" x2="144.78" y2="106.68" width="0.1524" layer="91"/>
+<label x="144.78" y="106.68" size="1.27" layer="95" rot="R180" xref="yes"/>
+<pinref part="R13" gate="G$1" pin="2"/>
+</segment>
+</net>
+<net name="NC_D5" class="0">
+<segment>
+<wire x1="152.4" y1="104.14" x2="144.78" y2="104.14" width="0.1524" layer="91"/>
+<label x="144.78" y="104.14" size="1.27" layer="95" rot="R180" xref="yes"/>
+<pinref part="R14" gate="G$1" pin="2"/>
+</segment>
+</net>
+<net name="NC_D3" class="0">
+<segment>
+<wire x1="152.4" y1="101.6" x2="144.78" y2="101.6" width="0.1524" layer="91"/>
+<label x="144.78" y="101.6" size="1.27" layer="95" rot="R180" xref="yes"/>
+<pinref part="R15" gate="G$1" pin="2"/>
 </segment>
 </net>
 <net name="NC_D1" class="0">
+<segment>
+<wire x1="152.4" y1="99.06" x2="144.78" y2="99.06" width="0.1524" layer="91"/>
+<label x="144.78" y="99.06" size="1.27" layer="95" rot="R180" xref="yes"/>
+<pinref part="R16" gate="G$1" pin="2"/>
+</segment>
+</net>
+<net name="N$10" class="0">
+<segment>
+<pinref part="SV2" gate="1" pin="11"/>
+<wire x1="187.96" y1="111.76" x2="195.58" y2="111.76" width="0.1524" layer="91"/>
+<pinref part="R17" gate="G$1" pin="2"/>
+</segment>
+</net>
+<net name="NC_D11_R" class="0">
+<segment>
+<pinref part="SV2" gate="1" pin="9"/>
+<wire x1="187.96" y1="109.22" x2="195.58" y2="109.22" width="0.1524" layer="91"/>
+<pinref part="R18" gate="G$1" pin="2"/>
+</segment>
+</net>
+<net name="NC_D6_R" class="0">
+<segment>
+<pinref part="SV2" gate="1" pin="7"/>
+<wire x1="187.96" y1="106.68" x2="195.58" y2="106.68" width="0.1524" layer="91"/>
+<pinref part="R19" gate="G$1" pin="2"/>
+</segment>
+</net>
+<net name="NC_D4_R" class="0">
+<segment>
+<pinref part="SV2" gate="1" pin="5"/>
+<wire x1="187.96" y1="104.14" x2="195.58" y2="104.14" width="0.1524" layer="91"/>
+<pinref part="R20" gate="G$1" pin="2"/>
+</segment>
+</net>
+<net name="NC_D2_R" class="0">
+<segment>
+<pinref part="SV2" gate="1" pin="3"/>
+<wire x1="187.96" y1="101.6" x2="195.58" y2="101.6" width="0.1524" layer="91"/>
+<pinref part="R21" gate="G$1" pin="2"/>
+</segment>
+</net>
+<net name="NC_D0_R" class="0">
+<segment>
+<pinref part="SV2" gate="1" pin="1"/>
+<wire x1="187.96" y1="99.06" x2="195.58" y2="99.06" width="0.1524" layer="91"/>
+<pinref part="R22" gate="G$1" pin="2"/>
+</segment>
+</net>
+<net name="N$22" class="0">
+<segment>
+<pinref part="SV1" gate="1" pin="6"/>
+<wire x1="172.72" y1="162.56" x2="165.1" y2="162.56" width="0.1524" layer="91"/>
+<pinref part="R23" gate="G$1" pin="1"/>
+</segment>
+</net>
+<net name="NC_A3_R" class="0">
+<segment>
+<pinref part="SV1" gate="1" pin="4"/>
+<wire x1="172.72" y1="160.02" x2="165.1" y2="160.02" width="0.1524" layer="91"/>
+<pinref part="R24" gate="G$1" pin="1"/>
+</segment>
+</net>
+<net name="NC_A1_R" class="0">
+<segment>
+<pinref part="SV1" gate="1" pin="2"/>
+<wire x1="172.72" y1="157.48" x2="165.1" y2="157.48" width="0.1524" layer="91"/>
+<pinref part="R25" gate="G$1" pin="1"/>
+</segment>
+</net>
+<net name="NC_A4_R" class="0">
+<segment>
+<pinref part="SV1" gate="1" pin="5"/>
+<wire x1="187.96" y1="162.56" x2="200.66" y2="162.56" width="0.1524" layer="91"/>
+<pinref part="R26" gate="G$1" pin="2"/>
+</segment>
+</net>
+<net name="NC_A2_R" class="0">
+<segment>
+<pinref part="SV1" gate="1" pin="3"/>
+<wire x1="187.96" y1="160.02" x2="200.66" y2="160.02" width="0.1524" layer="91"/>
+<pinref part="R27" gate="G$1" pin="2"/>
+</segment>
+</net>
+<net name="NC_A0_R" class="0">
+<segment>
+<pinref part="SV1" gate="1" pin="1"/>
+<wire x1="187.96" y1="157.48" x2="200.66" y2="157.48" width="0.1524" layer="91"/>
+<pinref part="R28" gate="G$1" pin="2"/>
+</segment>
+</net>
+<net name="NC_D12_R" class="0">
+<segment>
+<pinref part="SV2" gate="1" pin="10"/>
+<wire x1="172.72" y1="109.22" x2="162.56" y2="109.22" width="0.1524" layer="91"/>
+<pinref part="R9" gate="G$1" pin="1"/>
+</segment>
+</net>
+<net name="NC_D1_R" class="0">
 <segment>
 <pinref part="SV2" gate="1" pin="2"/>
@@
 </segment>
 </net>
-<net name="NC_D3" class="0">
+<net name="NC_D3_R" class="0">
 <segment>
 <pinref part="SV2" gate="1" pin="4"/>
@@
 </segment>
 </net>
-<net name="ND_D5" class="0">
-<segment>
-<pinref part="SV2" gate="1" pin="6"/>
-<wire x1="172.72" y1="104.14" x2="162.56" y2="104.14" width="0.1524" layer="91"/>
-<pinref part="R14" gate="G$1" pin="1"/>
-</segment>
-</net>
-<net name="NC_D7" class="0">
+<net name="NC_D7_R" class="0">
 <segment>
 <pinref part="SV2" gate="1" pin="8"/>
@@
 <net name="NC_D12" class="0">
 <segment>
-<pinref part="SV2" gate="1" pin="10"/>
-<wire x1="172.72" y1="109.22" x2="162.56" y2="109.22" width="0.1524" layer="91"/>
-<pinref part="R9" gate="G$1" pin="1"/>
-</segment>
-</net>
-<net name="NC_D11" class="0">
-<segment>
-<label x="218.44" y="109.22" size="1.27" layer="95" xref="yes"/>
-<wire x1="205.74" y1="109.22" x2="218.44" y2="109.22" width="0.1524" layer="91"/>
-<pinref part="R18" gate="G$1" pin="1"/>
-</segment>
-</net>
-<net name="N$1" class="0">
-<segment>
-<pinref part="SV2" gate="1" pin="12"/>
-<wire x1="172.72" y1="111.76" x2="162.56" y2="111.76" width="0.1524" layer="91"/>
-<pinref part="R7" gate="G$1" pin="1"/>
-</segment>
-</net>
-<net name="N$2" class="0">
-<segment>
 <wire x1="152.4" y1="109.22" x2="144.78" y2="109.22" width="0.1524" layer="91"/>
 <label x="144.78" y="109.22" size="1.27" layer="95" rot="R180" xref="yes"/>
 <pinref part="R9" gate="G$1" pin="2"/>
-</segment>
-</net>
-<net name="N$5" class="0">
-<segment>
-<wire x1="152.4" y1="106.68" x2="144.78" y2="106.68" width="0.1524" layer="91"/>
-<label x="144.78" y="106.68" size="1.27" layer="95" rot="R180" xref="yes"/>
-<pinref part="R13" gate="G$1" pin="2"/>
-</segment>
-</net>
-<net name="N$6" class="0">
-<segment>
-<wire x1="152.4" y1="104.14" x2="144.78" y2="104.14" width="0.1524" layer="91"/>
-<label x="144.78" y="104.14" size="1.27" layer="95" rot="R180" xref="yes"/>
-<pinref part="R14" gate="G$1" pin="2"/>
-</segment>
-</net>
-<net name="N$8" class="0">
-<segment>
-<wire x1="152.4" y1="101.6" x2="144.78" y2="101.6" width="0.1524" layer="91"/>
-<label x="144.78" y="101.6" size="1.27" layer="95" rot="R180" xref="yes"/>
-<pinref part="R15" gate="G$1" pin="2"/>
-</segment>
-</net>
-<net name="N$9" class="0">
-<segment>
-<wire x1="152.4" y1="99.06" x2="144.78" y2="99.06" width="0.1524" layer="91"/>
-<label x="144.78" y="99.06" size="1.27" layer="95" rot="R180" xref="yes"/>
-<pinref part="R16" gate="G$1" pin="2"/>
-</segment>
-</net>
-<net name="N$10" class="0">
-<segment>
-<pinref part="SV2" gate="1" pin="11"/>
-<wire x1="187.96" y1="111.76" x2="195.58" y2="111.76" width="0.1524" layer="91"/>
-<pinref part="R17" gate="G$1" pin="2"/>
-</segment>
-</net>
-<net name="N$11" class="0">
-<segment>
-<pinref part="SV2" gate="1" pin="9"/>
-<wire x1="187.96" y1="109.22" x2="195.58" y2="109.22" width="0.1524" layer="91"/>
-<pinref part="R18" gate="G$1" pin="2"/>
-</segment>
-</net>
-<net name="N$12" class="0">
-<segment>
-<pinref part="SV2" gate="1" pin="7"/>
-<wire x1="187.96" y1="106.68" x2="195.58" y2="106.68" width="0.1524" layer="91"/>
-<pinref part="R19" gate="G$1" pin="2"/>
-</segment>
-</net>
-<net name="N$17" class="0">
-<segment>
-<pinref part="SV2" gate="1" pin="5"/>
-<wire x1="187.96" y1="104.14" x2="195.58" y2="104.14" width="0.1524" layer="91"/>
-<pinref part="R20" gate="G$1" pin="2"/>
-</segment>
-</net>
-<net name="N$18" class="0">
-<segment>
-<pinref part="SV2" gate="1" pin="3"/>
-<wire x1="187.96" y1="101.6" x2="195.58" y2="101.6" width="0.1524" layer="91"/>
-<pinref part="R21" gate="G$1" pin="2"/>
-</segment>
-</net>
-<net name="N$21" class="0">
-<segment>
-<pinref part="SV2" gate="1" pin="1"/>
-<wire x1="187.96" y1="99.06" x2="195.58" y2="99.06" width="0.1524" layer="91"/>
-<pinref part="R22" gate="G$1" pin="2"/>
-</segment>
-</net>
-<net name="N$22" class="0">
-<segment>
-<pinref part="SV1" gate="1" pin="6"/>
-<wire x1="172.72" y1="162.56" x2="165.1" y2="162.56" width="0.1524" layer="91"/>
-<pinref part="R23" gate="G$1" pin="1"/>
-</segment>
-</net>
-<net name="N$23" class="0">
-<segment>
-<pinref part="SV1" gate="1" pin="4"/>
-<wire x1="172.72" y1="160.02" x2="165.1" y2="160.02" width="0.1524" layer="91"/>
-<pinref part="R24" gate="G$1" pin="1"/>
-</segment>
-</net>
-<net name="N$24" class="0">
-<segment>
-<pinref part="SV1" gate="1" pin="2"/>
-<wire x1="172.72" y1="157.48" x2="165.1" y2="157.48" width="0.1524" layer="91"/>
-<pinref part="R25" gate="G$1" pin="1"/>
-</segment>
-</net>
-<net name="N$25" class="0">
-<segment>
-<pinref part="SV1" gate="1" pin="5"/>
-<wire x1="187.96" y1="162.56" x2="200.66" y2="162.56" width="0.1524" layer="91"/>
-<pinref part="R26" gate="G$1" pin="2"/>
-</segment>
-</net>
-<net name="N$26" class="0">
-<segment>
-<pinref part="SV1" gate="1" pin="3"/>
-<wire x1="187.96" y1="160.02" x2="200.66" y2="160.02" width="0.1524" layer="91"/>
-<pinref part="R27" gate="G$1" pin="2"/>
-</segment>
-</net>
-<net name="N$27" class="0">
-<segment>
-<pinref part="SV1" gate="1" pin="1"/>
-<wire x1="187.96" y1="157.48" x2="200.66" y2="157.48" width="0.1524" layer="91"/>
-<pinref part="R28" gate="G$1" pin="2"/>
 </segment>
 </net>
@@
 </sheet>
 </sheets>
+<errors>
+</errors>
 </schematic>
 </drawing>
