File: Landing Gear Layout.brd (EAGLE design)
At the start: 60 x 50 mm, 48 parts, among them J1 3x2 M, J2 S2B-PH-SM4-TB(LF)(SN), J3 629105136821, SW1 AYZ0202AGRLC, SW2 !RESET, U1 MCP73831, U2 MIC5219, U3 ATMEGA32U4-AUR, X2 16 MHz

Commit message: Add files via upload
Moved everything to MASTER branch
Parts:
- added SERV_MOTOR1, SERV_MOTOR3: (no value), con-lstb:MA03-1
- moved C2 0.22 mm to (34.3, 26.6)
Connections:
- net 3.3V3: now also SERV_MOTOR1.2, SERV_MOTOR3.2
- net GND: now also SERV_MOTOR1.1, SERV_MOTOR3.1
- net GND1: now also SERV_MOTOR1.3, SERV_MOTOR3.3
Routing:
- net GND1: track 0.00 -> 53.6 mm
- net GND: track 0.00 -> 43.2 mm
- net 3.3V3: track 0.00 -> 40.5 mm
- net 3.3V: track 104.6 -> 115.8 mm
- net VBUS: track 67.1 -> 68.0 mm
